Commit message: WIP: Arduino integration and joint standardization - pushing for cross-platform development

File: homeplus_urdf/urdf/homeplus_urdf.urdf (robot description, URDF)
Before this commit: robot homeplus_urdf, 16 links, 15 joints
Links:
- link Arm1: mass 0.142552966932564 -> 0.142458692227375
- link Arm2: mass 0.116259676580817 -> 0.116165417113753
- link FingerL: mass 0.025246070206814 -> 0.00826272704561505
- link FingerR: mass 0.025246070206814 -> 0.00654686444828128
- link Frame: mass 2.00952337404394 -> 3.29967833042039
- link Hand: mass 0.0151490486204883 -> 0.0198930486204883
- link Telescope: mass 0.252043575649992 -> 0.251949294795669
- link WheelFR: mass 0.0242299260398931 -> 0.024229926039893
- link Wrist: mass 0.0363561056351058 -> 0.036356105635106
- link base: mass 1.36547736598414 -> 1.93599733287841
Joints:
- joint JointArm1: limit lower=-4.8 upper=0.436 effort=1 velocity=1 -> lower=-3.229 upper=0 effort=1 velocity=1; origin xyz=0 0.027951 0.19359 rpy=0 0 0 -> xyz=0 0.027951 0.52359 rpy=0 0 0
- joint JointArm2: limit lower=-2.967 upper=2.269 effort=1 velocity=1 -> lower=-2.932 upper=1.274 effort=1 velocity=1; origin xyz=0.1879 0.0665 -0.40296 rpy=0 0 0 -> xyz=0 0.0665 -0.44462 rpy=0 0 0
- joint JointFingerL: axis -0.25882 0 0.96593 -> 0 0 1; limit lower=0 upper=1.396 effort=1 velocity=1 -> lower=-0.262 upper=1.396 effort=1 velocity=1; origin xyz=0.07403 -0.0115 0.040542 rpy=0 0 0 -> xyz=0.076 -0.012 0.025 rpy=0 0 0
- joint JointFingerR: axis -0.25882 0 0.96593 -> 0 0 -1; limit lower=-1.396 upper=0 effort=1 velocity=1 -> lower=-0.262 upper=1.396 effort=1 velocity=1; mimic joint=JointFingerL multiplier=-1 offset=0 -> joint=JointFingerL multiplier=1 offset=0; origin xyz=0.07403 -0.0365 0.040542 rpy=0 0 0 -> xyz=0.076 -0.036 0.025 rpy=0 0 0
- joint JointFrame: limit lower=-0.085 upper=0 effort=1 velocity=1 -> lower=-0.15 upper=0 effort=1 velocity=1
- joint JointHand: limit lower=0 upper=2.967 effort=1 velocity=1 -> lower=-1.309 upper=1.571 effort=1 velocity=1; origin xyz=-0.0026339 0.035169 -0.01502 rpy=0 0 0 -> xyz=0.0125 0.035169 -0.008735 rpy=0 0 0
- joint JointTelescope: limit lower=-0.1 upper=0.115 effort=1 velocity=1 -> lower=-0.43 upper=0 effort=1 velocity=1
- joint JointWheelBR: axis 0.70711 0.70711 0 -> 0.707106781186548 0.707106781186547 0; origin xyz=-0.19308 -0.19308 -0.033 rpy=0 0 0 -> xyz=-0.193081475451951 -0.193081475451951 -0.033 rpy=0 0 0
- joint JointWrist: axis -0.42262 0 0.90631 -> 1 0 0; limit lower=0 upper=5.236 effort=1 velocity=1 -> lower=-1.396 upper=1.396 effort=1 velocity=1; origin xyz=0.16059 -0.0175 -0.40102 rpy=0 0 0 -> xyz=0.43131 -0.0175 -0.023935 rpy=0 0 0

Commit message: Sync joint limits, URDF, and Arduino output; standardize start state

File: homeplus_urdf/urdf/homeplus_urdf.urdf (robot description, URDF)
Before this commit: robot homeplus_urdf, 16 links, 15 joints
Links:
- link Arm1: mass 0.142458692227375 -> 0.142458692559679
- link Arm2: mass 0.116165417113753 -> 0.116165387072632
- link FingerL: mass 0.00826272704561505 -> 0.00826272704567777
- link FingerR: mass 0.00654686444828128 -> 0.00654686444830018
- link Hand: mass 0.0198930486204883 -> 0.0198930486204882
- link Telescope: mass 0.251949294795669 -> 0.251949298778275
- link Wrist: mass 0.036356105635106 -> 0.0363561056351056
Joints:
- joint JointArm1: axis 0 1 0 -> 0 -1 0; limit lower=-3.229 upper=0 effort=1 velocity=1 -> lower=-0.7854 upper=2.4435 effort=1 velocity=1; origin xyz=0 0.027951 0.52359 rpy=0 0 0 -> xyz=0 0.027951 0.093587 rpy=0 0 0
- joint JointArm2: axis 0 1 0 -> 0 -1 0; limit lower=-2.932 upper=1.274 effort=1 velocity=1 -> lower=-1.274 upper=2.932 effort=1 velocity=1; origin xyz=0 0.0665 -0.44462 rpy=0 0 0 -> xyz=0.31439 0.0665 -0.31439 rpy=0 0 0
- joint JointFingerL: axis 0 0 1 -> 0.70711 0 0.70711; limit lower=-0.262 upper=1.396 effort=1 velocity=1 -> lower=0 upper=1.5708 effort=1 velocity=1; origin xyz=0.076 -0.012 0.025 rpy=0 0 0 -> xyz=0.071418 -0.012 -0.036062 rpy=0 0 0
- joint JointFingerR: axis 0 0 -1 -> -0.70711 0 -0.70711; limit lower=-0.262 upper=1.396 effort=1 velocity=1 -> lower=0 upper=1.5708 effort=1 velocity=1; origin xyz=0.076 -0.036 0.025 rpy=0 0 0 -> xyz=0.071418 -0.036 -0.036062 rpy=0 0 0
- joint JointFrame: axis 0 0 -1 -> 0 0 1; limit lower=-0.15 upper=0 effort=1 velocity=1 -> lower=0 upper=0.15 effort=1 velocity=1
- joint JointHand: axis 0 1 0 -> 0 -1 0; limit lower=-1.309 upper=1.571 effort=1 velocity=1 -> lower=-1.571 upper=1.309 effort=1 velocity=1; origin xyz=0.0125 0.035169 -0.008735 rpy=0 0 0 -> xyz=0.0026623 0.035169 -0.015015 rpy=0 0 0
- joint JointTelescope: limit lower=-0.43 upper=0 effort=1 velocity=1 -> lower=0 upper=0.43 effort=1 velocity=1
- joint JointWrist: axis 1 0 0 -> 0.70711 0 -0.70711; origin xyz=0.43131 -0.0175 -0.023935 rpy=0 0 0 -> xyz=0.28806 -0.0175 -0.32191 rpy=0 0 0

Commit message: push

File: homeplus_urdf/urdf/homeplus_urdf.urdf (robot description, URDF)
Before this commit: robot homeplus_urdf, 16 links, 15 joints
Links:
- added link camera_color_optical_frame
- added link camera_depth_optical_frame
- added link camera_link
Joints:
- added joint JointCameraColorOptical: type fixed, parent camera_link, child camera_color_optical_frame, origin xyz=0 0 0 rpy=-1.57079632679 0 -1.57079632679
- added joint JointCameraDepthOptical: type fixed, parent camera_link, child camera_depth_optical_frame, origin xyz=0 0 0 rpy=-1.57079632679 0 -1.57079632679
- added joint JointCameraMount: type fixed, parent Hand, child camera_link, origin xyz=0.06 -0.02 0.03 rpy=0 0 0
