Commit message: Fix coffee pickup execution
- enforce level gripper orientation
- correct grip timing and Arduino control
- update camera and OctoMap integration

File: homeplus_urdf_description/urdf/homeplus_urdf.xacro (robot description, xacro)
@@ -188,4 +188,13 @@
   </collision>
 </link>
+<!-- Tool-center point used for Cartesian goals. This is an initial CAD-based
+     estimate at the front center of the gripper; calibrate xyz against the
+     physical finger contact point if higher grasp accuracy is required. -->
+<link name="grasp_tcp"/>
+<joint name="palm_to_grasp_tcp" type="fixed">
+  <parent link="palm_1"/>
+  <child link="grasp_tcp"/>
+  <origin xyz="0.105 -0.026 -0.027" rpy="0 0 0"/>
+</joint>
 <link name="FingerL_new_1">
   <inertial>
@@ -422,4 +431,5 @@
 </joint>
 <joint name="rear_camera_to_base" type="fixed">
+  <!-- Keep the exported camera mesh in the original rear body opening. -->
   <origin xyz="-0.17907 0.0 0.2794" rpy="0 0 0"/>
   <parent link="base_link"/>
@@ -428,5 +438,7 @@
 <link name="rear_camera_link"/>
 <joint name="rear_camera_link_alias" type="fixed">
-  <origin xyz="0 0 0" rpy="0 0 3.141592653589793"/>
+  <!-- The physical sensor moved to the left face while the legacy CAD mesh
+       remains at the rear opening. This frame is the actual sensor pose. -->
+  <origin xyz="0.17907 0.17907 0" rpy="0 0 1.5707963267948966"/>
   <parent link="rear_camera_link_1"/>
   <child link="rear_camera_link"/>

Commit message: feat: integrate multi-camera perception and safer task execution
- add MolmoPoint detection and target-filtered obstacle clouds
- improve pickup/button planning and Arduino acknowledgments
- update launch configs, scripts, and documentation

File: homeplus_urdf_description/urdf/homeplus_urdf.xacro (robot description, xacro)
@@ -195,5 +195,18 @@
   <parent link="palm_1"/>
   <child link="grasp_tcp"/>
-  <origin xyz="0.105 -0.026 -0.027" rpy="0 0 0"/>
+  <!-- CAD geometry puts the physical gripper forward axis about 20 degrees
+       downward from palm +X.  Positive pitch aligns grasp_tcp +X with that
+       axis, so a world RPY goal of 0 0 0 is horizontal to the ground. -->
+  <origin xyz="0.105 -0.026 -0.027" rpy="0 0.349066 0"/>
+</joint>
+<!-- Contact frame for single-finger button pressing. Its X/Y position starts
+     from the CAD forward surface at joint_grip_L=70 degrees; the Z coordinate
+     includes the measured 3 cm downward shift to the lower physical finger.
+     Button tasks using it must command and hold the gripper at 70 degrees. -->
+<link name="press_tcp"/>
+<joint name="grasp_tcp_to_press_tcp" type="fixed">
+  <parent link="grasp_tcp"/>
+  <child link="press_tcp"/>
+  <origin xyz="0.07735 0.02253 -0.04204" rpy="0 0 0"/>
 </joint>
 <link name="FingerL_new_1">
